Commit message: updated dynamixel motor logic

File: arm.urdf (robot description, URDF)
Before this commit: robot arm, 5 links, 4 joints
Links:
- link lowerarm: geometry visual box size=20.0 1.0 1.0
- link upperarm: geometry visual box size=20.0 1.0 1.0
Joints:
- joint base_to_upperarm: limit lower=0.0 upper=6.283 effort=1000.0 velocity=0.5 -> lower=-3.1416 upper=3.1416 effort=1000.0 velocity=0.5
- joint lowerarm_to_wrist: limit lower=-1.571 upper=1.571 effort=1000.0 velocity=0.5 -> lower=-3.1416 upper=3.1416 effort=1000.0 velocity=0.5; origin xyz=5.0 0.0 0.0 rpy=0.0 0.0 0.0 -> xyz=20.0 0.0 0.0 rpy=0.0 0.0 0.0
- joint upperarm_to_lowerarm: limit lower=0.0 upper=6.283 effort=1000.0 velocity=0.5 -> lower=-3.1416 upper=3.1416 effort=1000.0 velocity=0.5; origin xyz=5.0 0.0 0.0 rpy=0.0 0.0 0.0 -> xyz=20.0 0.0 0.0 rpy=0.0 0.0 0.0
- joint wrist_to_grip: limit lower=-1.571 upper=1.571 effort=1000.0 velocity=0.5 -> lower=-3.1416 upper=3.1416 effort=1000.0 velocity=0.5
